File: Hardware/2.8in touch display hat/2.8in touch display hat.kicad_sch (KiCad schematic)
At the start: 53 parts, among them J1 B2B (JST-SH), J2 LRA (PicoBlade), Q1 NMOS, U1 DRV2605LDGS, U2 MMC5603NJ, U3 VEML7700-TR, U4 ATECC608B

Commit message: hat
Parts:
- added C20, C21, C22: 100nF, Capacitor_SMD:C_0603_1608Metric, symbol Device:C_Small
- added D11, D12, D13: WS2812B-2020, LED_SMD:LED_WS2812B-2020_PLCC4_2.0x2.0mm, symbol LED:WS2812B-2020
- C13, C15, C18: footprint Capacitor_SMD:C_1206_3216Metric -> Capacitor_SMD:C_0603_1608Metric
Connections:
- net +3.3V: now also C20.1, C21.1, C22.1, D11.4 (VDD), D12.4 (VDD), D13.4 (VDD)
- net GND: now also C20.2, C21.2, C22.2, D11.2 (VSS), D12.2 (VSS), D13.2 (VSS)
- net LRA+: now reaches J2.1 (Pin_1), U1.7 (OUT+)
- net LRA-: now reaches J2.2 (Pin_2), U1.9 (OUT-)
- net at D10.1 (DOUT): now also D11.3 (DIN)
- new net: D11.1 (DOUT), D12.3 (DIN)
- new net: D12.1 (DOUT), D13.3 (DIN)
- no-connect marks 2 -> 5
Other:
- moved on the sheet: ANT1, ANT2, C1, C10, C11, C12, C13, C14, C15, C16, C17, C18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
