File: Hardware/2.8in touch display hat/2.8in touch display hat.kicad_pcb (KiCad board)
At the start: 2 copper layers, 50 x 69 mm, 53 parts, among them J1 B2B (JST-SH), J2 LRA (PicoBlade), Q1 NMOS, U1 DRV2605LDGS, U3 VEML7700-TR, U4 ATECC608B

Commit message: PCB R1.5
Parts:
- added TP1: +3.3V, TestPoint:TestPoint_Pad_D1.0mm, B.Cu at (162.2, 131.6)
- added TP2: VBUS, TestPoint:TestPoint_Pad_D1.0mm, B.Cu at (164.4, 131.6)
- added TP3: SCL, TestPoint:TestPoint_Pad_D1.0mm, B.Cu at (160.1, 131.6)
- added TP4: SDA, TestPoint:TestPoint_Pad_D1.0mm, B.Cu at (157.9, 131.6)
- added TP5: LEDS, TestPoint:TestPoint_Pad_D1.0mm, B.Cu at (153.6, 131.6)
- added TP6: CHARGE, TestPoint:TestPoint_Pad_D1.0mm, B.Cu at (155.8, 131.6)
- added U2: MMC5603NJ, EasyEDA:FLIPCHIP-4_L0.8-W0.8-R2-C2-P0.40-TL, F.Cu at (143.9, 118.2)
- moved G*** 21.9 mm to (134.8, 130.0)
Routing:
- net +3.3V: track 60.7 -> 75.8 mm
- net GND: track 69.5 -> 54.5 mm, vias 45 -> 40
- net /SDA: track 25.7 -> 32.0 mm, vias 2 -> 3
- net /SCL: track 27.7 -> 33.1 mm, vias 0 -> 1
- net /CHARGE: track 14.9 -> 20.1 mm, vias 2 -> 3
- net VBUS: track 12.4 -> 15.8 mm, vias 0 -> 1
- net /GPIO15: track 24.2 -> 27.3 mm, vias 0 -> 3
Other:
- board text added: "Multi-function Hat For: Waveshare 2.8{dblquote} Touch ESP32"
